File: devices/tape/hardware/tape.kicad_sch (KiCad schematic)
At the start: 26 parts, among them J1 SPEAKER_OUT, M1 Motor_DC, Q1 BC337, U1 NE5532, U2 LM386

Commit message: fix(tape): rename kicad projet
Parts:
- added C10: 10u, symbol Device:C_Polarized
- added C2: 10u, symbol Device:C
- added R10: 1k, symbol Device:R
- added R11: 1k5, symbol Device:R
- added U3: LM1117T-ADJ, Package_TO_SOT_THT:TO-220-3_Horizontal_TabDown, symbol Regulator_Linear:LM1117T-ADJ
Connections:
- net 3V: now also C10.1, R10.1, U3.2 (VO)
- net GND: now also C10.2, C2.2, R11.2
- new net: R10.2, R11.1, U3.1 (ADJ)
- new net 5V: C2.1, U3.3 (VI)
Other:
- note added: "* or trimmer for exact 3V"
- note added: "AMP"
- note added: "PAM8403"
- moved on the sheet: C1, C3, C4, C5, C6, C7, C8, C9, D1, FB1, J1, M1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
